File: electronica/cad/_prueba_mcp/prueba_mcp.kicad_pcb (KiCad board)
At the start: 2 copper layers, 0 parts

Commit message: electronica: PCB editada en vivo con Konnect por la API de KiCad (ELE-027)
- Actualizar PCB desde esquema, contorno, mover huellas, rutear y guardar
  por la API; DRC sin cortocircuitos y Gerbers generados.
- La API solo responde si KiCad se abre desde el menú Inicio: con doble
  clic en el proyecto el canal desaparece al cerrarse la primera instancia.
  Regla de arranque agregada al flujo KiCad.
- .history/ de KiCad 10 en .gitignore.

Co-Authored-By: Claude Opus 5.5 <noreply@anthropic.com>
Parts:
- added J1: ENTRADA, Connector_PinHeader_2.54mm:PinHeader_1x02_P2.54mm_Vertical, F.Cu at (106.0, 92.0)
- added R1: 10k, Resistor_THT:R_Axial_DIN0207_L6.3mm_D2.5mm_P7.62mm_Horizontal, F.Cu at (115.0, 88.0)
- added R2: 10k, Resistor_THT:R_Axial_DIN0207_L6.3mm_D2.5mm_P7.62mm_Horizontal, F.Cu at (115.0, 100.0)
Routing:
- net /NODO_A: track 0.00 -> 13.0 mm
Other:
- board outline added: 40 x 30 mm
