File: electronica/cad/_prueba_mcp/prueba_mcp.kicad_sch (KiCad schematic)
At the start: 3 parts, among them J1 ENTRADA

Commit message: electronica: PCB editada en vivo con Konnect por la API de KiCad (ELE-027)
- Actualizar PCB desde esquema, contorno, mover huellas, rutear y guardar
  por la API; DRC sin cortocircuitos y Gerbers generados.
- La API solo responde si KiCad se abre desde el menú Inicio: con doble
  clic en el proyecto el canal desaparece al cerrarse la primera instancia.
  Regla de arranque agregada al flujo KiCad.
- .history/ de KiCad 10 en .gitignore.

Co-Authored-By: Claude Opus 5.5 <noreply@anthropic.com>
Parts:
- J1: footprint (none) -> Connector_PinHeader_2.54mm:PinHeader_1x02_P2.54mm_Vertical
- R1, R2: footprint (none) -> Resistor_THT:R_Axial_DIN0207_L6.3mm_D2.5mm_P7.62mm_Horizontal
Changed lines of the file:
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@@
 			)
 		)
-		(property "Footprint" ""
+		(property "Footprint" "Connector_PinHeader_2.54mm:PinHeader_1x02_P2.54mm_Vertical"
 			(at 59.69 80.01 0)
 			(hide yes)
@@
 			)
 		)
-		(property "Footprint" ""
+		(property "Footprint" "Resistor_THT:R_Axial_DIN0207_L6.3mm_D2.5mm_P7.62mm_Horizontal"
 			(at 100.33 69.85 0)
 			(hide yes)
@@
 			)
 		)
-		(property "Footprint" ""
+		(property "Footprint" "Resistor_THT:R_Axial_DIN0207_L6.3mm_D2.5mm_P7.62mm_Horizontal"
 			(at 100.33 100.33 0)
 			(hide yes)
