File: electronica/cad/segway_base/segway_base.kicad_pcb (KiCad board)
At the start: 2 copper layers, 0 parts

Commit message: electronica: esquema v0.4 simplificado y PCB v0.1 en curso (pausa)
- Especificación v0.4: 60 componentes y 47 nets para placa casera
  (sin puntos de prueba ni alternativas no montadas); ERC 0 y netlist igual.
- Huellas de los 7 módulos en segway_modulos.pretty.
- Reglas de fabricación casera, 71 supuestos (supuestos.md / .json).
- Constructor de PCB construir_pcb.py y flujo guardado; placa a medio
  rutear. Instrucciones de reanudación en estado_actual.md (ELE-032).

Co-Authored-By: Claude Opus 5.5 <noreply@anthropic.com>
Parts:
- added A1: Blue Pill STM32F103C8T6, segway_modulos:ROB-012_BluePill_STM32F103C8_40p, F.Cu at (114.3, 73.7)
- added A2: GY-521 MPU6050 0x68, segway_modulos:ROB-013_MPU6050_modulo_8p, F.Cu at (73.7, 94.0)
- added A3: DRV8871 mód. IZQ (enchufable), segway_modulos:ROB-008_DRV8871_modulo_8p, F.Cu at (45.7, 58.4)
- added A4: DRV8871 mód. DER (prov., enchufable), segway_modulos:ROB-008_DRV8871_modulo_8p, F.Cu at (96.5, 58.4)
- added A5: INA219 MCU-219 0x41 IZQ, segway_modulos:ROB-002_INA219_MCU-219_8p, F.Cu at (61.0, 55.9)
- added A6: INA219 MCU-219 0x44 DER, segway_modulos:ROB-002_INA219_MCU-219_8p, F.Cu at (111.8, 55.9)
- added A7: INA226 0x40 lógica+bus, segway_modulos:ROB-009_INA226_modulo_8p, F.Cu at (40.6, 73.7)
- added A8: Mini buck 5V ROB-006, segway_modulos:ROB-005-006_MiniBuck_modulo_4p, F.Cu at (58.4, 106.7)
- added A9: Mini buck 3,3V ROB-005 (3V3_PER), segway_modulos:ROB-005-006_MiniBuck_modulo_4p, F.Cu at (48.3, 96.5)
- added C1: 470µ/35V low-ESR, Capacitor_THT:CP_Radial_D10.0mm_P5.00mm, F.Cu at (144.8, 58.4)
- added C14: 100n/50V cerámico de disco (104), Capacitor_THT:C_Disc_D5.0mm_W2.5mm_P5.00mm, F.Cu at (137.2, 111.8)
- added C3: 10µ/50V X7R multicapa radial, Capacitor_THT:C_Disc_D7.5mm_W5.0mm_P5.00mm, F.Cu at (147.3, 68.6)
- added C4: 47µ/35V low-ESR, Capacitor_THT:CP_Radial_D6.3mm_P2.50mm, F.Cu at (50.8, 30.5)
- added C5: 47µ/35V low-ESR, Capacitor_THT:CP_Radial_D6.3mm_P2.50mm, F.Cu at (101.6, 30.5)
- added C8: 470µ/16V low-ESR, Capacitor_THT:CP_Radial_D8.0mm_P3.50mm, F.Cu at (88.9, 111.8)
- added C9: 470µ/16V low-ESR, Capacitor_THT:CP_Radial_D8.0mm_P3.50mm, F.Cu at (104.1, 106.7)
- added D1: SA15A (alt. P6KE18A), Diode_THT:D_DO-15_P10.16mm_Horizontal, F.Cu at (147.3, 73.7)
- added D2: 1N5819, Diode_THT:D_DO-41_SOD81_P10.16mm_Horizontal, F.Cu at (106.7, 114.3)
- added D3: BZX79-C12, Diode_THT:D_DO-35_SOD27_P7.62mm_Horizontal, F.Cu at (152.4, 61.0)
- added D4: LED rojo 3mm VM, LED_THT:LED_D3.0mm, F.Cu at (137.2, 83.8)
- added F1: ATO 15A lento, Fuse:Fuseholder_Blade_ATO_Littelfuse_Pudenz_2_Pin, F.Cu at (167.6, 48.3)
- added F2: ATM 4A, Fuse:Fuseholder_Blade_Mini_Keystone_3568, F.Cu at (144.8, 43.2)
- added F3: ATM 4A, Fuse:Fuseholder_Blade_Mini_Keystone_3568, F.Cu at (144.8, 35.6)
- added F4: ATM 7,5A, Fuse:Fuseholder_Blade_Mini_Keystone_3568, F.Cu at (152.4, 94.0)
- added F5: ATM 1A, Fuse:Fuseholder_Blade_Mini_Keystone_3568, F.Cu at (144.8, 50.8)
- added H1: M3, MountingHole:MountingHole_3.2mm_M3, F.Cu at (29.4, 29.4)
- added H2: M3, MountingHole:MountingHole_3.2mm_M3, F.Cu at (181.4, 29.4)
- added H3: M3, MountingHole:MountingHole_3.2mm_M3, F.Cu at (29.4, 121.4)
- added H4: M3, MountingHole:MountingHole_3.2mm_M3, F.Cu at (181.4, 121.4)
- added J1: Batería MKDS3 1=P− 2=P+, TerminalBlock_Phoenix:TerminalBlock_Phoenix_MKDS-3-2-5.08_1x02_P5.08mm_Horizontal, F.Cu at (180.3, 53.3)
- added J11: Motor IZQ 1=M+ 2=M−, TerminalBlock_Phoenix:TerminalBlock_Phoenix_MKDS-1,5-2-5.08_1x02_P5.08mm_Horizontal, F.Cu at (43.2, 30.5)
- added J12: Motor DER 1=M+ 2=M−, TerminalBlock_Phoenix:TerminalBlock_Phoenix_MKDS-1,5-2-5.08_1x02_P5.08mm_Horizontal, F.Cu at (94.0, 30.5)
- added J13: Servo IZQ JR, Connector_PinHeader_2.54mm:PinHeader_1x03_P2.54mm_Vertical, F.Cu at (81.3, 101.6)
- added J14: Servo DER JR, Connector_PinHeader_2.54mm:PinHeader_1x03_P2.54mm_Vertical, F.Cu at (101.6, 96.5)
- added J15: UBEC entrada, TerminalBlock_Phoenix:TerminalBlock_Phoenix_MKDS-1,5-2-5.08_1x02_P5.08mm_Horizontal, F.Cu at (172.7, 101.6)
- added J16: UBEC salida 6V PT1,5 1=GND 2=V+, TerminalBlock_Phoenix:TerminalBlock_Phoenix_PT-1,5-2-3.5-H_1x02_P3.50mm_Horizontal, F.Cu at (86.4, 121.9)
- added J18: Voltímetro ROB-004, TerminalBlock_Phoenix:TerminalBlock_Phoenix_PT-1,5-3-3.5-H_1x03_P3.50mm_Horizontal, F.Cu at (35.6, 121.9)
- added J23: UART1 1=GND 2=TX 3=RX, Connector_PinHeader_2.54mm:PinHeader_1x03_P2.54mm_Vertical, F.Cu at (106.7, 88.9)
- added J3: Lazo interruptor+paro, TerminalBlock_Phoenix:TerminalBlock_Phoenix_MKDS-3-2-5.08_1x02_P5.08mm_Horizontal, F.Cu at (154.9, 48.3)
- added J4: Paro MPT0,5 1=GND 2=PARO (NC), TerminalBlock_Phoenix:TerminalBlock_Phoenix_MPT-0,5-2-2.54_1x02_P2.54mm_Horizontal, F.Cu at (104.1, 76.2)
- added J7: Encoder IZQ PT1,5 1=GND 2=A 3=B 4=V, TerminalBlock_Phoenix:TerminalBlock_Phoenix_PT-1,5-4-3.5-H_1x04_P3.50mm_Horizontal, F.Cu at (137.2, 121.9)
- added J8: Encoder DER PT1,5 1=GND 2=A 3=B 4=V, TerminalBlock_Phoenix:TerminalBlock_Phoenix_PT-1,5-4-3.5-H_1x04_P3.50mm_Horizontal, F.Cu at (96.5, 121.9)
- added Q1: IRF4905, Package_TO_SOT_THT:TO-220-3_Vertical, F.Cu at (157.5, 66.0)
- added R1: 2k2 1%, Resistor_THT:R_Axial_DIN0207_L6.3mm_D2.5mm_P10.16mm_Horizontal, F.Cu at (83.8, 63.5)
- added R13: 10k, Resistor_THT:R_Axial_DIN0207_L6.3mm_D2.5mm_P10.16mm_Horizontal, F.Cu at (157.5, 111.8)
- added R14: 10k, Resistor_THT:R_Axial_DIN0207_L6.3mm_D2.5mm_P10.16mm_Horizontal, F.Cu at (162.6, 111.8)
- added R15: 10k, Resistor_THT:R_Axial_DIN0207_L6.3mm_D2.5mm_P10.16mm_Horizontal, F.Cu at (86.4, 96.5)
- added R16: 10k, Resistor_THT:R_Axial_DIN0207_L6.3mm_D2.5mm_P10.16mm_Horizontal, F.Cu at (96.5, 99.1)
- added R2: 2k2 1%, Resistor_THT:R_Axial_DIN0207_L6.3mm_D2.5mm_P10.16mm_Horizontal, F.Cu at (83.8, 68.6)
- added R22: 100k 1%, Resistor_THT:R_Axial_DIN0207_L6.3mm_D2.5mm_P10.16mm_Horizontal, F.Cu at (147.3, 88.9)
- added R23: 12k 1%, Resistor_THT:R_Axial_DIN0207_L6.3mm_D2.5mm_P10.16mm_Horizontal, F.Cu at (137.2, 106.7)
- added R24: 10k, Resistor_THT:R_Axial_DIN0207_L6.3mm_D2.5mm_P10.16mm_Horizontal, F.Cu at (114.3, 66.0)
- added R28: 5k1, Resistor_THT:R_Axial_DIN0207_L6.3mm_D2.5mm_P10.16mm_Horizontal, F.Cu at (152.4, 78.7)
- added R29: 10k, Resistor_THT:R_Axial_DIN0207_L6.3mm_D2.5mm_P10.16mm_Horizontal, F.Cu at (162.6, 66.0)
- added R3: 2k2 1%, Resistor_THT:R_Axial_DIN0207_L6.3mm_D2.5mm_P10.16mm_Horizontal, F.Cu at (142.2, 101.6)
- added R35: 4k7 1%, Resistor_THT:R_Axial_DIN0207_L6.3mm_D2.5mm_P10.16mm_Horizontal, F.Cu at (71.1, 66.0)
- added R36: 4k7 1%, Resistor_THT:R_Axial_DIN0207_L6.3mm_D2.5mm_P10.16mm_Horizontal, F.Cu at (71.1, 71.1)
- added R37: 4k7 1%, Resistor_THT:R_Axial_DIN0207_L6.3mm_D2.5mm_P10.16mm_Horizontal, F.Cu at (101.6, 63.5)
- added R38: 4k7 1%, Resistor_THT:R_Axial_DIN0207_L6.3mm_D2.5mm_P10.16mm_Horizontal, F.Cu at (99.1, 68.6)
- added R4: 2k2 1%, Resistor_THT:R_Axial_DIN0207_L6.3mm_D2.5mm_P10.16mm_Horizontal, F.Cu at (137.2, 101.6)
- added R5: 1k 1%, Resistor_THT:R_Axial_DIN0207_L6.3mm_D2.5mm_P10.16mm_Horizontal, F.Cu at (86.4, 83.8)
- added R6: 1k 1%, Resistor_THT:R_Axial_DIN0207_L6.3mm_D2.5mm_P10.16mm_Horizontal, F.Cu at (96.5, 81.3)
- added R7: 10k, Resistor_THT:R_Axial_DIN0207_L6.3mm_D2.5mm_P10.16mm_Horizontal, F.Cu at (91.4, 83.8)
- added R8: 10k, Resistor_THT:R_Axial_DIN0207_L6.3mm_D2.5mm_P10.16mm_Horizontal, F.Cu at (101.6, 81.3)
Routing:
- net /VM_LOG_F: track 0.00 -> 141.0 mm
- net /GND: track 0.00 -> 130.1 mm
- net /VM_IZQ_F: track 0.00 -> 77.0 mm
- net /VM_BUS: track 0.00 -> 62.5 mm
- net /VM_DER: track 0.00 -> 44.4 mm
- net /VM_IZQ: track 0.00 -> 44.4 mm
- net /VM_DER_F: track 0.00 -> 19.9 mm
- net /VBAT_F: track 0.00 -> 19.0 mm
- net /VM_UBEC: track 0.00 -> 13.9 mm
- net /VBAT_P: track 0.00 -> 12.7 mm
- net /MOT_DER_1: track 0.00 -> 12.3 mm
- net /MOT_IZQ_1: track 0.00 -> 12.3 mm
- net /MOT_DER_2: track 0.00 -> 11.4 mm
- net /MOT_IZQ_2: track 0.00 -> 11.4 mm
- net /VBAT_SW: track 0.00 -> 8.81 mm
Other:
- board outline added: 160 x 100 mm
- rule pad_to_mask_clearance: 0.05 -> 0
