File: electronica/cad/segway_base/segway_base.kicad_sch (KiCad schematic)
At the start: 58 parts, among them J1 Batería MKDS3 1=P− 2=P+, J11 Motor IZQ 1=M+ 2=M−, J12 Motor DER 1=M+ 2=M−, J13 Servo IZQ JR, J14 Servo DER JR, J15 UBEC entrada, J16 UBEC salida 6V PT1,5 1=GND 2=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, J18 Voltímetro ROB-004, J3 Lazo interruptor+paro, J4 Paro MPT0,5 1=GND 2=PARO (NC), J7 Encoder IZQ PT1,5 1=GND 2=A 3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, J8 Encoder DER PT1,5 1=GND 2=A 3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, Q1 IRF4905

Commit message: electronica: pines reasignados por geometría y constructor de PCB con Freerouting JAR y puentes (ELE-032)
- IN de los drivers en GPIO4-7 y encoders en GPIO15-18 (SUP-28); esquema
  regenerado con ERC 0 y netlist coincidente.
- construir_pcb.py: Freerouting 2.5.0 en JAR con Java 25 (la versión nativa
  se cae con zonas prohibidas) y conversión de tramos superiores en
  puentes de alambre. Ubicación para la ESP32-S3 en revisión.

Co-Authored-By: Claude Opus 5.5 <noreply@anthropic.com>
Connections:
- net ENC_DER_A: now also A1.8 (GPIO15); no longer A1.6 (GPIO6)
- net ENC_DER_B: now also A1.9 (GPIO16); no longer A1.7 (GPIO7)
- net ENC_IZQ_A: now also A1.10 (GPIO17); no longer A1.4 (GPIO4)
- net ENC_IZQ_B: now also A1.11 (GPIO18); no longer A1.5 (GPIO5)
- net IN1_DER_MCU: now also A1.4 (GPIO4); no longer A1.10 (GPIO17)
- net IN1_IZQ_MCU: now also A1.6 (GPIO6); no longer A1.8 (GPIO15)
- net IN2_DER_MCU: now also A1.5 (GPIO5); no longer A1.11 (GPIO18)
- net IN2_IZQ_MCU: now also A1.7 (GPIO7); no longer A1.9 (GPIO16)
