File: electronica/cad/segway_potencia/segway_potencia.kicad_sch (KiCad schematic)
At the start: 48 parts, among them J1 Batería MKDS3 1=P− 2=P+, J11 Motor IZQ 1=M+ 2=M−, J12 Motor DER 1=M+ 2=M−, J13 Servo IZQ JR, J14 Servo DER JR, J15 UBEC entrada, J16 UBEC salida 6V PT1,5 1=GND 2=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, J18 Voltímetro ROB-004, J20 Cable lógica-potencia 2x8, J3 Lazo interruptor+paro, Q1 IRF4905

Commit message: electronica: PCB v0.1 de la placa de lógica, una cara, DRC limpio (ELE-032)
- Ruteo a mano por topología (agente/placas/logica.py, TEC-04): DRC 0 errores,
  0 sin conectar, 0 de paridad; 2 puentes de alambre (3V3 17,8 mm y GND 7,6 mm).
- Mapa de GPIO y cable J20 elegidos por geometría: columna par del IDC en línea
  con A1.15-22; SCL/SDA pasan por el MPU. D2 pasa a la placa de potencia (5V_MCU
  por el cable); J7 con extremos invertidos. Esquemas de lógica y potencia
  regenerados: ERC 0 y netlist coincidente.
- construir_pcb.py con --placa y --fabricar: puentes fijos, áreas sin relleno,
  rótulos y escala en cobre, relleno con reglas reales, PDF 1:1, taladros.
- Supuestos SUP-04/15/24/26/28 cambiados y SUP-72 a SUP-74 nuevos.

Co-Authored-By: Claude Opus 5.5 <noreply@anthropic.com>
Parts:
- added D2: 1N5819, Diode_THT:D_DO-41_SOD81_P10.16mm_Horizontal, symbol Diode:1N5819
Connections:
- net 3V3_MCU: now also J20.9 (Pin_9); no longer J20.5 (Pin_5)
- net 5V: now also D2.2 (A); no longer J20.2 (Pin_2), J20.4 (Pin_4)
- net GND: now also J20.11 (Pin_11), J20.15 (Pin_15), J20.16 (Pin_16); no longer J20.1 (Pin_1), J20.3 (Pin_3), J20.7 (Pin_7)
- net I2C_SCL: now also J20.7 (Pin_7); no longer J20.8 (Pin_8)
- net I2C_SDA: now also J20.5 (Pin_5); no longer J20.6 (Pin_6)
- net IN1_DER_MCU: now also J20.2 (Pin_2); no longer J20.11 (Pin_11)
- net IN1_IZQ_MCU: now also J20.6 (Pin_6); no longer J20.13 (Pin_13)
- net IN2_DER_MCU: now also J20.4 (Pin_4); no longer J20.12 (Pin_12)
- net IN2_IZQ_MCU: now also J20.8 (Pin_8); no longer J20.14 (Pin_14)
- net INA_ALERT: now also J20.1 (Pin_1); no longer J20.9 (Pin_9)
- net SERVO_DER_MCU: now also J20.12 (Pin_12); no longer J20.16 (Pin_16)
- net SERVO_IZQ_MCU: now also J20.10 (Pin_10); no longer J20.15 (Pin_15)
- net VBAT_ADC: now also J20.3 (Pin_3); no longer J20.10 (Pin_10)
- new net 5V_MCU: D2.1 (K), J20.13 (Pin_13), J20.14 (Pin_14)

Commit message: electronica: PCB v0.1 de la placa de potencia, una cara, DRC limpio (ELE-032)
- Placa de potencia 150 x 110 mm: barra VM_BUS, lomo GND en estrella entre los
  pads de los fusibles, ramas por canal de motor, franja de servos y banda
  lógica. DRC 0 errores, 0 sin conectar, 0 de paridad; 7 puentes fijos.
- Ruteo híbrido (TEC-05): esqueleto y bus I2C a mano (J20 -> A7 -> A5 ->
  corredor bajo los módulos -> A6), Freerouting solo para nets simples, vías
  prohibidas sobre componentes y poda automática de puentes redundantes.
- Cable J20 y GPIO reordenados por geometría (VBAT en GPIO3, ALERT en GPIO8,
  columna par servos/IN); placa de lógica regenerada y re-verificada (0/0/0).
- J20.11 sin conexión en la potencia; INA226 sin separador opcional.
- Supuestos SUP-04/15/24/28/72 actualizados y SUP-75 a SUP-77 nuevos.

Co-Authored-By: Claude Opus 5.5 <noreply@anthropic.com>
Connections:
- net GND: no longer J20.11 (Pin_11)
- net IN1_DER_MCU: now also J20.8 (Pin_8); no longer J20.2 (Pin_2)
- net IN1_IZQ_MCU: now also J20.12 (Pin_12); no longer J20.6 (Pin_6)
- net IN2_DER_MCU: now also J20.6 (Pin_6); no longer J20.4 (Pin_4)
- net IN2_IZQ_MCU: now also J20.10 (Pin_10); no longer J20.8 (Pin_8)
- net INA_ALERT: now also J20.3 (Pin_3); no longer J20.1 (Pin_1)
- net SERVO_DER_MCU: now also J20.4 (Pin_4); no longer J20.12 (Pin_12)
- net SERVO_IZQ_MCU: now also J20.2 (Pin_2); no longer J20.10 (Pin_10)
- net VBAT_ADC: now also J20.1 (Pin_1); no longer J20.3 (Pin_3)
- no-connect marks 0 -> 1

Commit message: electronica: rótulos de cobre, revisión independiente y control eléctrico (ELE-039)
- Rótulos de polaridad y de fusibles en el cobre de las dos placas,
  ubicados con ubicar_rotulos.py sin partir el relleno GND (SUP-14).
- Revisión independiente del conexionado contra las fichas: módulos,
  cable, polaridades y niveles correctos. Riesgos nuevos: A7 y A8 entran
  girados y queman (SUP-80), aleta de Q1 con tensión (SUP-20), I2C junto
  a PWM en el cable (SUP-81).
- auditoria_electrica.py: control repetible del sistema (cable, pines
  críticos, 5 V lejos de la ESP32, módulos girados, I2C, cuellos de
  pista, niveles). Informe: 0 fallas, 6 avisos.
- J26 reordenado con GND en el medio; textos de la Blue Pill en la
  especificación corregidos.
- ERC 0 y netlist coincidente; DRC 0/0/0 en las dos placas; salidas de
  fabricación regeneradas.

Co-Authored-By: Claude Opus 5.5 <noreply@anthropic.com>
Parts:
- A7: Estado provisorio [H] (orden [V]; dirección de fábrica 0x40 [H], sujeta a aprobar el cambio del contrato §4.1; ubicación en la rama lógica = propuesta [H] que se desvía de [ENERGIA] §5.2 (INA226 en el bus), pendiente de Matías, REQ-14; unión VBS-IN− interna pendiente E-01; la 1x08 no tiene pin libre para codificar: invertido lleva VM_LOG_F a VCC (6 V abs.) y deja el shunt entre 3V3_PER y GND, así que la huella lleva un tope mecánico contra el cuerpo invertido y el contorno serigrafiado) | v0.4: huella segway_modulos:ROB-009_INA226_modulo_8p con tope NPTH de 3,2 mm (M3x16) contra la inserción invertida; ALERT con pull-up interna de PB13 (R21 eliminada, SUP-71); JP8 eliminado (SUP-67) -> provisorio [H] (orden [V]; dirección de fábrica 0x40 [H], sujeta a aprobar el cambio del contrato §4.1; ubicación en la rama lógica = propuesta [H] que se desvía de [ENERGIA] §5.2 (INA226 en el bus), pendiente de Matías, REQ-14; unión VBS-IN− interna pendiente E-01; la 1x08 no tiene pin libre para codificar: invertido lleva VM_LOG_F a VCC (6 V abs.) y deja el shunt entre 3V3_MCU y GND, así que la huella lleva un tope mecánico contra el cuerpo invertido y el contorno serigrafiado) | v0.4: huella segway_modulos:ROB-009_INA226_modulo_8p con tope NPTH de 3,2 mm (M3x16) contra la inserción invertida; ALERT con pull-up interna de GPIO8 (R21 eliminada, SUP-71); JP8 eliminado (SUP-67) | v0.6: sin el tope NPTH (caía sobre el bus I2C, SUP-75): se puede enchufar invertido. Rótulo VCC en el cobre junto al pin 8; si el equipo lo aprueba, se suelda directo en lugar de ir en zócalo (ELE-039)
- A8: Estado pendiente de medida [H]: mini buck de 5 V, chip no identificado (SUP-37); huella segway_modulos:ROB-005-006_MiniBuck_modulo_4p con pads supuestos en un rectángulo de 19,0 × 14,0 mm; validar en E-02; girado 180° une VM_LOG con 5V por la masa del módulo, así que en la v0.1 va girado 90° respecto de A9 y con rótulo 5V en cobre (SUP-38); A10 (LM2596 de respaldo) eliminado (SUP-63); C23 y C24 eliminados (SUP-69) -> pendiente de medida [H]: mini buck de 5 V, chip no identificado (SUP-37); huella segway_modulos:ROB-005-006_MiniBuck_modulo_4p con pads supuestos en un rectángulo de 19,0 × 14,0 mm; validar en E-02; girado 180° une VM_LOG con 5V por la masa del módulo, así que en la v0.1 va girado 90° respecto de A9 y con rótulo 5V en cobre (SUP-38); A10 (LM2596 de respaldo) eliminado (SUP-63); C23 y C24 eliminados (SUP-69) | v0.6: A9 eliminado, la codificación por giro ya no aplica. Rótulo IN+ en el cobre junto al pin 1; si el equipo lo aprueba, se suelda directo en lugar de ir en zócalo (ELE-039)
- C14: Fuente [DS-STM32] p.75 Ecuación 1 (carga del capacitor de muestreo de 8 pF); τ = 1,07 ms; huella THT de KiCad 10.0.7 (DEC-14, SUP-16) -> [DS-STM32] p.75 Ecuación 1 (carga del capacitor de muestreo de 8 pF); τ = 1,07 ms; huella THT de KiCad 10.0.7 (DEC-14, SUP-16) | v0.6: las referencias al STM32 ([DS-STM32], [RM0008]) son de la v0.3; la controladora es la ESP32-S3 (DEC-16)
- F5: Estado provisorio [H]: ATM de 1 A (SUP-49, propuesta 17), acota la falla de un regulador enchufado girado; verificar en E-02 que no abre con la carga de las entradas de A8/A9 (C24 eliminado, SUP-69) -> provisorio [H]: ATM de 1 A (SUP-49, propuesta 17), acota la falla de un regulador enchufado girado; verificar en E-02 que no abre con la carga de las entrada de A8 (C24 eliminado, SUP-69)
- R1: Fuente [DS-STM32] p.61 Tabla 36 (RPU 30-50 kΩ, fuga ±1 µA); [RM0008] §7.1.1 (Rev 6) p.99 (entrada flotante al reset); [DS-DRV] p.5 (RPD 100 kΩ, VIL 0,5 V); huella THT de KiCad 10.0.7 (DEC-14, SUP-16) -> [DS-STM32] p.61 Tabla 36 (RPU 30-50 kΩ, fuga ±1 µA); [RM0008] §7.1.1 (Rev 6) p.99 (entrada flotante al reset); [DS-DRV] p.5 (RPD 100 kΩ, VIL 0,5 V); huella THT de KiCad 10.0.7 (DEC-14, SUP-16) | v0.6: las referencias al STM32 ([DS-STM32], [RM0008]) son de la v0.3; la controladora es la ESP32-S3 (DEC-16)
- R22: Fuente [DS-STM32] p.74 Tabla 47 (rango 0 a VREF+ = VDDA en LQFP48), p.75 Tabla 48 (RAIN ≤ 25,2 kΩ con 28,5 ciclos); [DS-SMAJ] p.2; huella THT de KiCad 10.0.7 (DEC-14, SUP-16) -> [DS-STM32] p.74 Tabla 47 (rango 0 a VREF+ = VDDA en LQFP48), p.75 Tabla 48 (RAIN ≤ 25,2 kΩ con 28,5 ciclos); [DS-SMAJ] p.2; huella THT de KiCad 10.0.7 (DEC-14, SUP-16) | v0.6: las referencias al STM32 ([DS-STM32], [RM0008]) son de la v0.3; la controladora es la ESP32-S3 (DEC-16)
- R35: Estado provisorio [H] (nueva, a ratificar: protege PA6 si un DRV88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 -> provisorio [H] (nueva, a ratificar: protege GPIO14 si un DR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; Fuente [DS-STM32] p.37 Tablas 6-7 (pin no FT: VIN abs. 4 V, inyección ±5 mA); [DS-DRV] p.4-5 (VIH 1,5 V, RPD 100 kΩ, pulso ≥ 800 ns); huella THT de KiCad 10.0.7 (DEC-14, SUP-16) -> [DS-STM32] p.37 Tablas 6-7 (pin no FT: VIN abs. 4 V, inyección ±5 mA); [DS-DRV] p.4-5 (VIH 1,5 V, RPD 100 kΩ, pulso ≥ 800 ns); huella THT de KiCad 10.0.7 (DEC-14, SUP-16) | v0.6: las referencias al STM32 ([DS-STM32], [RM0008]) son de la v0.3; la controladora es la ESP32-S3 (DEC-16)
- R36: Estado provisorio [H] (nueva; protege PA7) | v0.4: THT: axial 1/4 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 -> provisorio [H] (nueva; protege GPIO13) | v0.4: THT: axial 1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
- R37: Estado provisorio [H] (nueva; protege PB0) | v0.4: THT: axial 1/4 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 -> provisorio [H] (nueva; protege GPIO12) | v0.4: THT: axial 1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
- R38: Estado provisorio [H] (nueva; protege PB1) | v0.4: THT: axial 1/4 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 -> provisorio [H] (nueva; protege GPIO11) | v0.4: THT: axial 1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
- R5: Fuente [ENERGIA] §2.2; [CONTRATO] §2.5; [DS-STM32] p.37 Tablas 6-7 (PA8 FT: VIN ≤ VDD + 4 V, inyección −5/+0 mA); [DS-STM32] Tabla 37 p.64 (niveles garantizados hasta 8 mA); huella THT de KiCad 10.0.7 (DEC-14, SUP-16) -> [ENERGIA] §2.2; [CONTRATO] §2.5; [DS-STM32] p.37 Tablas 6-7 (PA8 FT: VIN ≤ VDD + 4 V, inyección −5/+0 mA); [DS-STM32] Tabla 37 p.64 (niveles garantizados hasta 8 mA); huella THT de KiCad 10.0.7 (DEC-14, SUP-16) | v0.6: las referencias al STM32 ([DS-STM32], [RM0008]) son de la v0.3; la controladora es la ESP32-S3 (DEC-16)
- R6: Fuente [ENERGIA] §2.2; [CONTRATO] §2.5; [DS-STM32] p.37 Tablas 6-7 (PB15 FT); [DS-STM32] Tabla 37 p.64 (niveles garantizados hasta 8 mA); huella THT de KiCad 10.0.7 (DEC-14, SUP-16) -> [ENERGIA] §2.2; [CONTRATO] §2.5; [DS-STM32] p.37 Tablas 6-7 (PB15 FT); [DS-STM32] Tabla 37 p.64 (niveles garantizados hasta 8 mA); huella THT de KiCad 10.0.7 (DEC-14, SUP-16) | v0.6: las referencias al STM32 ([DS-STM32], [RM0008]) son de la v0.3; la controladora es la ESP32-S3 (DEC-16)
- R7: Fuente [RM0008] §7.1.1 (Rev 6) p.99 (PA8 flotante al reset); huella THT de KiCad 10.0.7 (DEC-14, SUP-16) -> [RM0008] §7.1.1 (Rev 6) p.99 (PA8 flotante al reset); huella THT de KiCad 10.0.7 (DEC-14, SUP-16) | v0.6: las referencias al STM32 ([DS-STM32], [RM0008]) son de la v0.3; la controladora es la ESP32-S3 (DEC-16)
- R8: Fuente [RM0008] §7.1.1 (Rev 6) p.99 (PB15 flotante al reset); huella THT de KiCad 10.0.7 (DEC-14, SUP-16) -> [RM0008] §7.1.1 (Rev 6) p.99 (PB15 flotante al reset); huella THT de KiCad 10.0.7 (DEC-14, SUP-16) | v0.6: las referencias al STM32 ([DS-STM32], [RM0008]) son de la v0.3; la controladora es la ESP32-S3 (DEC-16)

Commit message: electronica: PCB v0.2 de las dos placas, auditada (ELE-040)
- J3 y J4 pasan a pads para soldar el cable del interruptor y del paro.
- Montaje: A1-A4 en zócalo, A5-A8 soldados (DEC-20). A1 codificada:
  pin 24 cortado y posición tapada (revisión independiente: entraba
  girada o corrida y se quemaba).
- auditoria_electrica.py prueba giros y corrimientos de los módulos
  enchufados; 0 fallas, 3 avisos.
- Rótulos ambiguos de fusibles y VCC quitados; continuidad del cable
  J20 antes de enchufar; precinto en J3.
- Documentación v0.2, lista de compras, fabricación en rev-0.2.
- ERC 0, netlist coincidente, DRC 0/0/0 en las dos placas.

Co-Authored-By: Claude Opus 5.5 <noreply@anthropic.com>
Parts:
- removed J3: Lazo interruptor+paro, TerminalBlock_Phoenix:TerminalBlock_Phoenix_MKDS-3-2-5.08_1x02_P5.08mm_Horizontal, symbol Connector:Screw_Terminal_01x02
- added J3: Interruptor+paro NC en serie, cable 1,5 mm² solda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, Connector_Wire:SolderWire-1.5sqmm_1x02_P6mm_D1.7mm_OD3mm, symbol Connector_Generic:Conn_01x02
Connections:
- net VBAT_F: now also J3.1 (Pin_1)
- net VBAT_SW: now also J3.2 (Pin_2)
